File: carte_bras_barillet/carte_bras_barillet/carte_bras_barillet.kicad_sch (KiCad schematic)
At the start: 24 parts, among them IC1 VNH7100BASTR, J1 Conn_01x02_Pin, J2 Conn_01x02_Pin, J3 RJ11, J5 Conn_01x06_Socket, Q1 PMOS, U1 MCP2515-xSO, U2 MCP2562-E-P

Commit message: carte bat
Parts:
- removed J3: RJ11, symbol RJ11:RJ11
- removed U1: MCP2515-xSO, Package_SO:SOIC-18W_7.5x11.6mm_P1.27mm, symbol Interface_CAN_LIN:MCP2515-xSO
- added J3: 110990030, symbol 110990030:110990030
- added U3: NUCLEO-F303K8, symbol NUCLEO-F303K8:NUCLEO-F303K8
Connections:
- net +5: now also J3.2, U3.4_1 (VIN)
- net DIR: now also U3.3_13 (PA11); no longer RZ1.17 (GP26)
- net GND: now also J3.1, U3.3_4 (GND_1), U3.4_2 (GND_2)
- net INA-1: now also U3.4_9 (PA4); no longer RZ1.6 (GP5)
- net INB-1: now also U3.4_11 (PA1); no longer RZ1.7 (GP6)
- net MS1: now also U3.4_6 (PA7); no longer RZ1.16 (GP15)
- net MS2: now also U3.4_7 (PA6); no longer RZ1.15 (GP14)
- net MS3: now also U3.4_8 (PA5); no longer RZ1.14 (GP13)
- net PWM1: now also U3.3_1 (PA9); no longer RZ1.10 (GP9)
- net SEL01: now also U3.4_12 (PA0); no longer RZ1.8 (GP7)
- net STEP: now also U3.3_5 (PA12); no longer RZ1.18 (GP27)
- net val-courant-a: now also U3.3_14 (PB5)
- net /ENABLE: now also U3.3_2 (PA10); no longer RZ1.19 (GP28)
- net /RESET: now also U3.4_10 (PA3); no longer RZ1.20 (GP29)
- net at U2.6 (CANL): now also J3.4
- net at U2.7 (CANH): now also J3.3
- net CL: no longer names the net of RZ1.2 (GP1)
- net MISO: no longer names the net of RZ1.5 (GP4)
- net MOSI: no longer names the net of RZ1.4 (GP3)
- net SCK: no longer names the net of RZ1.3 (GP2)
