File: carte_moteur/carte hacheur.kicad_sch (KiCad schematic)
At the start: 32 parts, among them IC1 VNH7100BASTR, IC2 VNH7100BASTR, J1 Conn_01x02_Pin, J2 Conn_01x02_Pin, J3 Conn_01x02_Pin, J4 Conn_01x02_Pin, Q1 PMOS, Q2 PMOS, U1 RP2040, U2 MCP2562-E-P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

Commit message: rp2040 zero
Parts:
- removed U1: RP2040, Package_DFN_QFN:QFN-56-1EP_7x7mm_P0.4mm_EP3.2x3.2mm, symbol MCU_RaspberryPi:RP2040
- added RZ1: RP2040-Zero, symbol rp2040-zero:RP2040-Zero
- R1, R11: value ? -> 1K
Connections:
- net +5: now also RZ1.22 (5V)
- net GND: now also RZ1.23 (GND)
- net val-courant-a: now also RZ1.17 (GP26)
- net val-courant-b: now also RZ1.18 (GP27)
- net INA-1: now reaches R3.1
- net INA-1: now also RZ1.6 (GP5)
- net INB-2: now reaches R8.1
- net INB-2: now also RZ1.9 (GP8)
- net PWM2: now reaches R9.2
- net PWM2: now also RZ1.11 (GP10)
- net PWM1: now reaches R6.2
- net PWM1: now also RZ1.10 (GP9)
- net SEL02: now reaches R10.2
- net SEL02: now also RZ1.15 (GP14)
- net SCK: now reaches U3.13 (SCK)
- net SCK: now also RZ1.3 (GP2)
- net MOSI: now reaches U3.14 (SI)
- net MOSI: now also RZ1.4 (GP3)
- net MISO: now reaches U3.15 (SO)
- net MISO: now also RZ1.5 (GP4)
- net CS: now reaches U3.16 (~{CS})
- net SEL01: now reaches R4.2
- net SEL01: now also RZ1.14 (GP13)
- net INB-1: now reaches R5.1
- net INB-1: now also RZ1.7 (GP6)
- net INA-2: now reaches R7.1
- net INA-2: now also RZ1.8 (GP7)
- new net CL: RZ1.2 (GP1)
Other:
- moved on the sheet: R10, R4

Commit message: 1
Parts:
- added J5: RJ25, symbol Connector:RJ25
- R1, R11: value 1K -> 900
Connections:
- net GND: now also J5.6
- net at U2.6 (CANL): now also J5.2
- net at U2.7 (CANH): now also J5.1
Changed lines of the file:
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@@
+    (stroke (width 0) (type default))
+  )
+  (wire (pts (xy 236.22 179.07) (xy 245.745 179.07))
+    (stroke (width 0) (type default))
+  )
+  (wire (pts (xy 236.22 182.245) (xy 236.22 179.07))
     (stroke (width 0) (type default))
   )
@@
     (stroke (width 0) (type default))
   )
+  (wire (pts (xy 239.395 187.325) (xy 239.395 181.61))
+    (stroke (width 0) (type default))
+  )
   (wire (pts (xy 94.615 68.58) (xy 123.19 68.58))
     (stroke (width 0) (type default))
@@
     (stroke (width 0) (type default))
   )
+  (wire (pts (xy 236.22 187.325) (xy 239.395 187.325))
+    (stroke (width 0) (type default))
+  )
   (wire (pts (xy 114.3 188.595) (xy 116.205 188.595))
     (stroke (width 0) (type default))
@@
   )
   (wire (pts (xy 177.8 61.595) (xy 165.735 61.595))
+    (stroke (width 0) (type default))
+  )
+  (wire (pts (xy 239.395 181.61) (xy 245.745 181.61))
     (stroke (width 0) (type default))
   )
@@
       (effects (font (size 1.27 1.27)) (justify left))
     )
-    (property "Value" "1K" (at 125.095 73.66 0)
+    (property "Value" "900" (at 125.095 73.66 0)
       (effects (font (size 1.27 1.27)) (justify left))
     )
@@
       (effects (font (size 1.27 1.27)) (justify left))
     )
-    (property "Value" "1K" (at 241.3 71.755 0)
+    (property "Value" "900" (at 241.3 71.755 0)
       (effects (font (size 1.27 1.27)) (justify left))
     )
@@
         (path "/f1c67e3e-f7e5-476e-af36-48fc43174252"
           (reference "#PWR015") (unit 1)
+        )
+      )
+    )
+  )
+  (symbol (lib_id "power:GND") (at 245.745 191.77 0) (unit 1)
+    (in_bom yes) (on_board yes) (dnp no) (fields_autoplaced)
+    (property "Reference" "#PWR024" (at 245.745 198.12 0)
+      (effects (font (size 1.27 1.27)) hide)
+    )
+    (property "Value" "GND" (at 245.745 196.85 0)
+      (effects (font (size 1.27 1.27)))
+    )
+    (property "Footprint" "" (at 245.745 191.77 0)
+      (effects (font (size 1.27 1.27)) hide)
+    )
+    (property "Datasheet" "" (at 245.745 191.77 0)
+      (effects (font (size 1.27 1.27)) hide)
+    )
+    (pin "1")
+    (instances
+      (project "carte hacheur"
+        (path "/f1c67e3e-f7e5-476e-af36-48fc43174252"
+          (reference "#PWR024") (unit 1)
         )
       )
@@
         )
       )
+    )
+  )
+  (symbol (lib_id "Connector:RJ25") (at 255.905 184.15 180) (unit 1)
+    (in_bom yes) (on_board yes) (dnp no) (fields_autoplaced)
+    (property "Reference" "J5" (at 265.43 184.15 0)
+      (effects (font (size 1.27 1.27)) (justify right))
+    )
+    (property "Value" "RJ25" (at 265.43 186.69 0)
+      (effects (font (size 1.27 1.27)) (justify right))
+    )
+    (property "Footprint" "" (at 255.905 184.785 90)
+      (effects (font (size 1.27 1.27)) hide)
+    )
+    (property "Datasheet" "~" (at 255.905 184.785 90)
+      (effects (font (size 1.27 1.27)) hide)
+    )
+    (pin "1")
+    (pin "2")
+    (pin "3")
+    (pin "4")
+    (pin "5")
+    (pin "6")
+    (instances
+      (project "carte hacheur"
+        (path "/f1c67e3e-f7e5-476e-af36-48fc43174252"
+          (reference "J5") (unit 1)
+        )
+      )

Commit message: modif
Parts:
- removed J4: Conn_01x02_Pin, symbol Connector:Conn_01x02_Pin
- removed J5: RJ25, symbol Connector:RJ25
- removed Q2: PMOS, symbol Simulation_SPICE:PMOS
- removed R14: 10k, symbol Device:R
- added J4: RJ11, symbol RJ11:RJ11
Connections:
- net +5: now also J4.5
- net GND: now also J4.6
- net at U2.6 (CANL): now also J4.2
- net at U2.7 (CANH): now also J4.1
Other:
- moved on the sheet: U2

Commit message: carte bat
Parts:
- removed D1: 6.8v, symbol Device:D_Zener
- removed J1: Conn_01x02_Pin, symbol Connector:Conn_01x02_Pin
- removed J4: RJ11, symbol RJ11:RJ11
- removed Q1: PMOS, symbol Simulation_SPICE:PMOS
- removed RZ1: RP2040-Zero, symbol rp2040-zero:RP2040-Zero
- removed U2: MCP2562-E-P, Package_DIP:DIP-8_W7.62mm, symbol Interface_CAN_LIN:MCP2562-E-P
- removed U3: MCP2515-xSO, Package_SO:SOIC-18W_7.5x11.6mm_P1.27mm, symbol Interface_CAN_LIN:MCP2515-xSO
- added J1, J4, J5, J6: 110990030, symbol 110990030:110990030
Connections:
- net SEL02 is gone; now on net SEL01: R10.2
- net GND: now also J1.1, J4.1, J5.1, J6.1; no longer R13.2
- net PWM1: now also J5.3
- net PWM2: now also J5.4
- net SEL01: now also R13.1
- net val-courant-a: now also J4.3
- net val-courant-b: now also J4.4
- new net: J4.2, R13.2
- new net +12V: J1.2
