File: carte batterie/carte batterie.kicad_sch (KiCad schematic)
At the start: 30 parts, among them IC1 TPS3711DDCT, IC2 TPS54531DDA, J1 Conn_01x02_Pin, J2 Conn_01x02_Pin, J3 Conn_01x01_Pin, J4 RJ11, Q1 SI3127DV-T1-GE3, U1 ATtiny1616-S

Commit message: cart bat modif
Parts:
- removed R8: 51 0.125W, Resistor_SMD:R_0805_2012Metric, symbol Device:R
Connections:
- net +12V: no longer C1.1, C2.1, C3.1, IC2.2 (VIN)
- net +5V: now also R7.1
- net +12VS: now reaches J2.2 (Pin_2), Q1.1 (D_1)
- net +12VS: now also C1.1, C2.1, C3.1, IC2.2 (VIN)
Changed lines of the file:
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@@
   (junction (at 172.085 157.48) (diameter 0) (color 0 0 0 0)
   )
+  (junction (at 53.34 27.305) (diameter 0) (color 0 0 0 0)
+  )
   (junction (at 133.985 116.205) (diameter 0) (color 0 0 0 0)
   )
-  (junction (at 53.34 27.305) (diameter 0) (color 0 0 0 0)
-  )
   (junction (at 139.7 27.305) (diameter 0) (color 0 0 0 0)
   )
@@
     (stroke (width 0) (type default))
   )
+  (wire (pts (xy 53.34 24.13) (xy 53.34 27.305))
+    (stroke (width 0) (type default))
+  )
   (wire (pts (xy 131.445 59.055) (xy 144.78 59.055))
     (stroke (width 0) (type default))
@@
     (stroke (width 0) (type default))
   )
+  (wire (pts (xy 53.34 27.305) (xy 68.58 27.305))
+    (stroke (width 0) (type default))
+  )
   (wire (pts (xy 140.335 106.045) (xy 140.335 92.075))
     (stroke (width 0) (type default))
@@
     (stroke (width 0) (type default))
   )
-  (wire (pts (xy 53.34 24.13) (xy 53.34 27.305))
-    (stroke (width 0) (type default))
-  )
   (wire (pts (xy 90.17 106.045) (xy 140.335 106.045))
     (stroke (width 0) (type default))
@@
     (stroke (width 0) (type default))
   )
+  (wire (pts (xy 139.7 41.275) (xy 146.685 41.275))
+    (stroke (width 0) (type default))
+  )
+  (wire (pts (xy 159.385 116.205) (xy 162.56 116.205))
+    (stroke (width 0) (type default))
+  )
+  (wire (pts (xy 95.25 142.24) (xy 95.25 134.62))
+    (stroke (width 0) (type default))
+  )
+  (wire (pts (xy 133.985 157.48) (xy 172.085 157.48))
+    (stroke (width 0) (type default))
+  )
+  (wire (pts (xy 103.505 116.205) (xy 133.985 116.205))
+    (stroke (width 0) (type default))
+  )
+  (wire (pts (xy 89.535 109.22) (xy 89.535 97.155))
+    (stroke (width 0) (type default))
+  )
+  (wire (pts (xy 75.565 129.54) (xy 103.505 129.54))
+    (stroke (width 0) (type default))
+  )
+  (wire (pts (xy 143.51 125.095) (xy 143.51 129.54))
+    (stroke (width 0) (type default))
+  )
+  (wire (pts (xy 151.765 149.86) (xy 146.05 149.86))
+    (stroke (width 0) (type default))
+  )
+  (wire (pts (xy 139.7 27.305) (xy 173.355 27.305))
+    (stroke (width 0) (type default))
+  )
+  (wire (pts (xy 190.5 111.76) (xy 186.69 111.76))
+    (stroke (width 0) (type default))
+  )
+  (wire (pts (xy 133.985 132.08) (xy 146.05 132.08))
+    (stroke (width 0) (type default))
+  )
+  (wire (pts (xy 142.875 36.195) (xy 146.685 36.195))
+    (stroke (width 0) (type default))
+  )
   (wire (pts (xy 37.465 27.305) (xy 53.34 27.305))
     (stroke (width 0) (type default))
   )
-  (wire (pts (xy 139.7 41.275) (xy 146.685 41.275))
-    (stroke (width 0) (type default))
-  )
-  (wire (pts (xy 159.385 116.205) (xy 162.56 116.205))
-    (stroke (width 0) (type default))
-  )
-  (wire (pts (xy 95.25 142.24) (xy 95.25 134.62))
-    (stroke (width 0) (type default))
-  )
-  (wire (pts (xy 133.985 157.48) (xy 172.085 157.48))
-    (stroke (width 0) (type default))
-  )
-  (wire (pts (xy 103.505 116.205) (xy 133.985 116.205))
-    (stroke (width 0) (type default))
-  )
-  (wire (pts (xy 89.535 109.22) (xy 89.535 97.155))
-    (stroke (width 0) (type default))
-  )
-  (wire (pts (xy 75.565 129.54) (xy 103.505 129.54))
-    (stroke (width 0) (type default))
-  )
-  (wire (pts (xy 143.51 125.095) (xy 143.51 129.54))
-    (stroke (width 0) (type default))
-  )
-  (wire (pts (xy 151.765 149.86) (xy 146.05 149.86))
-    (stroke (width 0) (type default))
-  )
-  (wire (pts (xy 139.7 27.305) (xy 173.355 27.305))
-    (stroke (width 0) (type default))
-  )
-  (wire (pts (xy 190.5 111.76) (xy 186.69 111.76))
-    (stroke (width 0) (type default))
-  )
-  (wire (pts (xy 133.985 132.08) (xy 146.05 132.08))
-    (stroke (width 0) (type default))
-  )
-  (wire (pts (xy 142.875 36.195) (xy 146.685 36.195))
-    (stroke (width 0) (type default))
-  )
-  (wire (pts (xy 53.34 27.305) (xy 68.58 27.305))
-    (stroke (width 0) (type default))
-  )
   (wire (pts (xy 131.445 69.215) (xy 146.05 69.215))
     (stroke (width 0) (type default))
@@
     (stroke (width 0) (type default))
   )
-  (wire (pts (xy 172.085 136.525) (xy 172.085 138.43))
-    (stroke (width 0) (type default))
-  )
   (wire (pts (xy 214.63 27.305) (xy 214.63 46.99))
     (stroke (width 0) (type default))
@@
     (stroke (width 0) (type default))
   )
-  (wire (pts (xy 172.085 146.05) (xy 172.085 147.955))
+  (wire (pts (xy 172.085 136.525) (xy 172.085 147.955))
     (stroke (width 0) (type default))
   )
@@
     )
   )
-  (global_label "+12V" (shape input) (at 57.785 129.54 180) (fields_autoplaced)
+  (global_label "+12VS" (shape input) (at 57.785 129.54 180) (fields_autoplaced)
     (effects (font (size 1.27 1.27)) (justify right))
-    (property "Intersheetrefs" "${INTERSHEET_REFS}" (at 49.7198 129.54 0)
+    (property "Intersheetrefs" "${INTERSHEET_REFS}" (at 48.5103 129.54 0)
       (effects (font (size 1.27 1.27)) (justify right) hide)
     )
@@
     (effects (font (size 1.27 1.27)) (justify left))
     (property "Intersheetrefs" "${INTERSHEET_REFS}" (at 174.2533 59.055 0)
+      (effects (font (size 1.27 1.27)) (justify left) hide)
+    )
+  )
+  (global_label "+12VS" (shape input) (at 214.63 46.99 0) (fields_autoplaced)
+    (effects (font (size 1.27 1.27)) (justify left))
+    (property "Intersheetrefs" "${INTERSHEET_REFS}" (at 223.9047 46.99 0)
       (effects (font (size 1.27 1.27)) (justify left) hide)
     )
@@
         )
       )
-    )
-  )
-  (symbol (lib_id "Device:R") (at 172.085 142.24 0) (unit 1)
-    (in_bom yes) (on_board yes) (dnp no) (fields_autoplaced)
-    (property "Reference" "R8" (at 173.99 140.97 0)
-      (effects (font (size 1.27 1.27)) (justify left))
-    )
-    (property "Value" "51     0.125W" (at 173.99 143.51 0)
-      (effects (font (size 1.27 1.27)) (justify left))
-    )
-    (property "Footprint" "Resistor_SMD:R_0805_2012Metric" (at 170.307 142.24 90)
-      (effects (font (size 1.27 1.27)) hide)
-    )
-    (property "Datasheet" "https://docs.rs-online.com/3b75/0900766b80d98b26.pdf" (at 172.085 142.24 0)
-      (effects (font (size 1.27 1.27)) hide)
-    )
-    (pin "1")
-    (pin "2")
-    (instances
-      (project "carte batterie"
-        (path "/8afff8df-3578-4f51-814d-4ef430aba141"
-          (reference "R8") (unit 1)
-        )
-      )
