File: carte batterie/carte_verma/carte batterie.kicad_sch (KiCad schematic)
At the start: 52 parts, among them IC1 TPS3711DDCT, IC2 TPS54531DDA, IC3 TPS54531DDA, J2 110990030, J3 110990030, J4 110990030, J5 110990030, J7 Screw_Terminal_01x02, J8 Screw_Terminal_01x02, Q1 SI3127DV-T1-GE3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

Commit message: cart bat modif
Parts:
- removed R10, R8: 51 0.125W, Resistor_SMD:R_0805_2012Metric, symbol Device:R
Connections:
- net +12V: no longer C1.1, C11.1, C12.1, C13.1, C2.1, C3.1, IC2.2 (VIN), IC3.2 (VIN)
- net +5V: now also R7.1
- net +5Vn2: now also R11.1
- net +12VS: now reaches J2.2, Q1.6 (D_4), R13.1, R15.1
- net +12VS: now also C1.1, C11.1, C12.1, C13.1, C2.1, C3.1, IC2.2 (VIN), IC3.2 (VIN)
Changed lines of the file:
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@@
     (stroke (width 0) (type default))
   )
-  (wire (pts (xy 168.91 228.6) (xy 168.91 230.505))
+  (wire (pts (xy 168.91 219.075) (xy 168.91 230.505))
     (stroke (width 0) (type default))
   )
@@
     (stroke (width 0) (type default))
   )
-  (wire (pts (xy 160.655 146.05) (xy 160.655 147.955))
+  (wire (pts (xy 160.655 146.05) (xy 160.655 157.48))
     (stroke (width 0) (type default))
   )
@@
     (stroke (width 0) (type default))
   )
-  (wire (pts (xy 160.655 155.575) (xy 160.655 157.48))
-    (stroke (width 0) (type default))
-  )
   (wire (pts (xy 38.1 55.88) (xy 53.34 55.88))
-    (stroke (width 0) (type default))
-  )
-  (wire (pts (xy 168.91 219.075) (xy 168.91 220.98))
     (stroke (width 0) (type default))
   )
@@
     )
   )
-  (global_label "+12V" (shape input) (at 46.355 139.065 180) (fields_autoplaced)
+  (global_label "+12VS" (shape input) (at 200.66 41.275 90) (fields_autoplaced)
+    (effects (font (size 1.27 1.27)) (justify left))
+    (property "Intersheetrefs" "${INTERSHEET_REFS}" (at 200.66 32.0003 90)
+      (effects (font (size 1.27 1.27)) (justify left) hide)
+    )
+  )
+  (global_label "+12VS" (shape input) (at 46.355 139.065 180) (fields_autoplaced)
     (effects (font (size 1.27 1.27)) (justify right))
-    (property "Intersheetrefs" "${INTERSHEET_REFS}" (at 38.2898 139.065 0)
+    (property "Intersheetrefs" "${INTERSHEET_REFS}" (at 37.0803 139.065 0)
       (effects (font (size 1.27 1.27)) (justify right) hide)
     )
@@
     )
   )
-  (global_label "+12V" (shape input) (at 54.61 212.09 180) (fields_autoplaced)
+  (global_label "+12VS" (shape input) (at 54.61 212.09 180) (fields_autoplaced)
     (effects (font (size 1.27 1.27)) (justify right))
-    (property "Intersheetrefs" "${INTERSHEET_REFS}" (at 46.5448 212.09 0)
+    (property "Intersheetrefs" "${INTERSHEET_REFS}" (at 45.3353 212.09 0)
       (effects (font (size 1.27 1.27)) (justify right) hide)
     )
@@
     )
   )
-  (symbol (lib_id "Device:R") (at 168.91 224.79 0) (unit 1)
-    (in_bom yes) (on_board yes) (dnp no) (fields_autoplaced)
-    (property "Reference" "R10" (at 170.815 223.52 0)
-      (effects (font (size 1.27 1.27)) (justify left))
-    )
-    (property "Value" "51     0.125W" (at 170.815 226.06 0)
-      (effects (font (size 1.27 1.27)) (justify left))
-    )
-    (property "Footprint" "Resistor_SMD:R_0805_2012Metric" (at 167.132 224.79 90)
-      (effects (font (size 1.27 1.27)) hide)
-    )
-    (property "Datasheet" "https://docs.rs-online.com/3b75/0900766b80d98b26.pdf" (at 168.91 224.79 0)
-      (effects (font (size 1.27 1.27)) hide)
-    )
-    (pin "1")
-    (pin "2")
-    (instances
-      (project "carte batterie"
-        (path "/8afff8df-3578-4f51-814d-4ef430aba141"
-          (reference "R10") (unit 1)
-        )
-      )
-    )
-  )
   (symbol (lib_id "power:GND") (at 167.005 206.375 0) (unit 1)
     (in_bom yes) (on_board yes) (dnp no) (fields_autoplaced)
@@
         )
       )
-    )
-  )
-  (symbol (lib_id "Device:R") (at 160.655 151.765 0) (unit 1)
-    (in_bom yes) (on_board yes) (dnp no) (fields_autoplaced)
-    (property "Reference" "R8" (at 162.56 150.495 0)
-      (effects (font (size 1.27 1.27)) (justify left))
-    )
-    (property "Value" "51     0.125W" (at 162.56 153.035 0)
-      (effects (font (size 1.27 1.27)) (justify left))
-    )
-    (property "Footprint" "Resistor_SMD:R_0805_2012Metric" (at 158.877 151.765 90)
-      (effects (font (size 1.27 1.27)) hide)
-    )
-    (property "Datasheet" "https://docs.rs-online.com/3b75/0900766b80d98b26.pdf" (at 160.655 151.765 0)
-      (effects (font (size 1.27 1.27)) hide)
-    )
-    (pin "1")
-    (pin "2")
-    (instances
-      (project "carte batterie"
-        (path "/8afff8df-3578-4f51-814d-4ef430aba141"
-          (reference "R8") (unit 1)
-        )
-      )

Commit message: pcb cart bat start
Parts:
- added D3: D, symbol Device:D
Connections:
- net +12V: now also D3.2 (A); no longer IC1.5 (VDD), Q1.4 (S), R1.1, R15.2
- new net: D3.1 (K), IC1.5 (VDD), Q1.4 (S), R1.1, R15.2
Changed lines of the file:
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@@
   (junction (at 166.37 125.73) (diameter 0) (color 0 0 0 0)
   )
+  (junction (at 68.58 27.305) (diameter 0) (color 0 0 0 0)
+  )
   (junction (at 191.77 50.165) (diameter 0) (color 0 0 0 0)
   )
@@
   (junction (at 56.515 146.685) (diameter 0) (color 0 0 0 0)
   )
-  (junction (at 68.58 27.305) (diameter 0) (color 0 0 0 0)
-  )
   (junction (at 140.335 159.385) (diameter 0) (color 0 0 0 0)
   )
@@
     (stroke (width 0) (type default))
   )
+  (wire (pts (xy 64.77 27.305) (xy 68.58 27.305))
+    (stroke (width 0) (type default))
+  )
   (wire (pts (xy 89.535 97.155) (xy 88.265 97.155))
     (stroke (width 0) (type default))
@@
     (stroke (width 0) (type default))
   )
+  (wire (pts (xy 53.34 27.305) (xy 57.15 27.305))
+    (stroke (width 0) (type default))
+  )
   (wire (pts (xy 261.62 125.095) (xy 261.62 127))
     (stroke (width 0) (type default))
@@
   )
   (wire (pts (xy 122.555 141.605) (xy 134.62 141.605))
-    (stroke (width 0) (type default))
-  )
-  (wire (pts (xy 53.34 27.305) (xy 68.58 27.305))
     (stroke (width 0) (type default))
   )
@@
         )
       )
+    )
+  )
+  (symbol (lib_id "Device:D") (at 60.96 27.305 180) (unit 1)
+    (in_bom yes) (on_board yes) (dnp no) (fields_autoplaced)
+    (property "Reference" "D3" (at 60.96 21.59 0)
+      (effects (font (size 1.27 1.27)))
+    )
+    (property "Value" "D" (at 60.96 24.13 0)
+      (effects (font (size 1.27 1.27)))
+    )
+    (property "Footprint" "" (at 60.96 27.305 0)
+      (effects (font (size 1.27 1.27)) hide)
+    )
+    (property "Datasheet" "~" (at 60.96 27.305 0)
+      (effects (font (size 1.27 1.27)) hide)
+    )
+    (property "Sim.Device" "D" (at 60.96 27.305 0)
+      (effects (font (size 1.27 1.27)) hide)
+    )
+    (property "Sim.Pins" "1=K 2=A" (at 60.96 27.305 0)
+      (effects (font (size 1.27 1.27)) hide)
+    )
+    (pin "1")
+    (pin "2")
+    (instances
+      (project "carte batterie"
+        (path "/8afff8df-3578-4f51-814d-4ef430aba141"
+          (reference "D3") (unit 1)
+        )
+      )
